Commit message: first

File: src/mini_mec_description/urdf/mini_mec_robot.urdf.xacro (robot description, xacro)
@@ -1,6 +1,8 @@
 <?xml version="1.0" ?>
 <robot name="mini_mec" xmlns:xacro="http://www.ros.org/wiki/xacro">
+    <!-- Include common properties and gazebo-specific configurations -->
     <xacro:include filename="common_properties.xacro"/>
     <xacro:include filename="mobile_base_gazebo.xacro"/>
+    <!-- Base link definition -->
     <link name="base_link">
         <visual>
@@ -21,10 +23,5 @@
         <xacro:box_inertia m="3.23" l="0.54" w="0.37" h="0.11" xyz="0 0 0.0975" rpy="0 0 0"/> <!-- l, w, h is 2x the value to fix inertia values-->
     </link>
-    <joint name="left_wheel_joint" type="continuous">
-        <origin xyz="-0.085 0.0975 0.0375" rpy="1.57 0 0"/>
-        <parent link="base_link"/>
-        <child link="left_wheel_link"/>
-        <axis xyz="0 0 1"/>
-    </joint>
+    <!-- Left wheel joint and link -->
     <link name="left_wheel_link">
         <visual>
@@ -45,4 +42,10 @@
         <xacro:cylinder_inertia m="0.18" r="0.075" h="0.06" xyz="0 0 0" rpy="0 0 0"/> <!-- r, h is 2x the visual to fix inertia values-->
     </link>
+    <joint name="left_wheel_joint" type="continuous">
+        <origin xyz="-0.085 0.0975 0.0375" rpy="1.57 0 0"/>
+        <parent link="base_link"/>
+        <child link="left_wheel_link"/>
+        <axis xyz="0 0 1"/>
+    </joint>
     <joint name="right_wheel_joint" type="continuous">
         <origin xyz="-0.085 -0.0975 0.0375" rpy="1.57 0 0"/>
@@ -117,3 +120,76 @@
         <xacro:cylinder_inertia m="0.18" r="0.075" h="0.06" xyz="0 0 0" rpy="0 0 0"/> <!-- r, h is 2x the visual to fix inertia values-->
     </link>
+    <link name="imu_link">
+        <xacro:box_inertia m="0.005" l="0.005" w="0.005" h="0.005" xyz="0 0 0.0975" rpy="0 0 0"/>
+        <visual>
+            <origin xyz="0 0 0.0850" rpy="0 0 0"/>
+            <geometry>
+                <box size="0.005 0.005 0.005"/>
+            </geometry>
+            <material name="black">
+                <color rgba="0 0 0 1"/>
+            </material>
+        </visual>
+        <collision>
+            <origin xyz="0 0 0.0850" rpy="0 0 0"/>
+            <geometry>
+                <box size="0.005 0.005 0.005"/>
+            </geometry>
+        </collision>
+    </link>
+    <joint name="imu_joint" type="fixed">
+        <parent link="base_link"/>
+        <child link="imu_link"/>
+        <origin xyz="0 0 0.0425" rpy="0 0 0"/>
+    </joint>
+    <!--
+    <link name="camera_link">
+        <visual>
+            <geometry>
+                <box size="0.02 0.05 0.025"/>
+            </geometry>
+            <material name="grey"/>
+            <collision>
+                <geometry>
+                    <box size="0.02 0.05 0.025"/>
+                </geometry>
+            </collision>
+            <inertial>
+                <xacro:box_inertia m="0.1" l="0.1" w="0.01" h="0.05" xyz="0 0 0" rpy="0 0 0"/>
+            </inertial>
+        </visual>
+    </link>
+    <joint name="base_camera_joint" type="fixed">
+        <parent link="base_link"/>
+        <child link="camera_link"/>
+        <origin xyz="0.110 0 0.1    375" rpy=" 0 0 0"/>
+    </joint>
+    -->
+    <link name="lidar_link">
+        <visual>
+            <origin xyz="0.035 0 0.0785" rpy="0 0 0"/>
+            <geometry>
+                <cylinder radius="0.035" length="0.065"/>
+            </geometry>
+            <material name="grey">
+                <color rgba="0.5 0.5 0.5 1"/>
+            </material>
+        </visual>
+        <collision>
+            <origin xyz="0.035 0 0.0785" rpy="0 0 0"/>
+            <geometry>
+                <cylinder radius="0.035" length="0.065"/>
+            </geometry>
+        </collision>
+        <inertial>
+            <origin xyz="0.035 0 0.0785" rpy="0 0 0"/>
+            <mass value="0.8"/>
+            <inertia ixx="0.002" ixy="0" ixz="0" iyy="0.002" iyz="0" izz="0.002"/>
+        </inertial>
+    </link>
+    <joint name="lidar_joint" type="fixed">
+        <parent link="base_link"/>
+        <child link="lidar_link"/>
+        <origin xyz="0.035 0 0.0785" rpy="0 0 0"/>
+    </joint>
 </robot>

File: src/mini_mec_description/urdf/mobile_base_gazebo.xacro (robot description, xacro)
@@ -26,3 +26,105 @@
           </plugin>
     </gazebo>
+    <gazebo reference="imu_link">
+        <sensor type="imu" name="imu_sensor">
+            <always_on>true</always_on>
+            <update_rate>100</update_rate>
+            <imu>
+                <angular_velocity>
+                    <x>
+                        <noise type="gaussian">
+                            <mean>0.0</mean>
+                            <stddev>2e-4</stddev>
+                        </noise>
+                    </x>
+                    <y>
+                        <noise type="gaussian">
+                            <mean>0.0</mean>
+                            <stddev>2e-4</stddev>
+                        </noise>
+                    </y>
+                    <z>
+                        <noise type="gaussian">
+                            <mean>0.0</mean>
+                            <stddev>2e-4</stddev>
+                        </noise>
+                    </z>
+                </angular_velocity>
+                <linear_acceleration>
+                    <x>
+                        <noise type="gaussian">
+                            <mean>0.0</mean>
+                            <stddev>1.7e-2</stddev>
+                        </noise>
+                    </x>
+                    <y>
+                        <noise type="gaussian">
+                            <mean>0.0</mean>
+                            <stddev>1.7e-2</stddev>
+                        </noise>
+                    </y>
+                    <z>
+                        <noise type="gaussian">
+                            <mean>0.0</mean>
+                            <stddev>1.7e-2</stddev>
+                        </noise>
+                    </z>
+                </linear_acceleration>
+            </imu>
+            <plugin name="imu" filename="libgazebo_ros_imu_sensor.so"/>
+        </sensor>
+    </gazebo>
+    <!--
+    <gazebo reference="camera_link">
+        <material>Gazebo/Red</material>
+        <sensor name="camera_sensor" type="camera">
+            <pose>0 0 0 0 0 0</pose>
+            <visualize>false</visualize>
+            <update_rate>30.0</update_rate>
+            <plugin name="camera_sensor" filename="libgazebo_ros_camera.so">
+                <frame_name>camera_link</frame_name>
+            </plugin>
+        </sensor>
+    </gazebo>
+    -->
+    <gazebo reference="lidar_link">
+        <sensor type="ray" name="lidar_sensor">
+            <always_on>true</always_on>
+            <update_rate>200</update_rate>
+            <ray>
+                <scan>
+                    <horizontal>
+                        <samples>720</samples>
+                        <resolution>1</resolution>
+                        <min_angle>-3.14159</min_angle>
+                        <max_angle>3.14159</max_angle>
+                    </horizontal>
+                    <vertical>
+                        <samples>200</samples>
+                        <resolution>1</resolution>
+                        <min_angle>0</min_angle>
+                        <max_angle>1.5707</max_angle>
+                    </vertical>
+                </scan>
+                <range>
+                    <min>0.2</min>
+                    <max>10.0</max>
+                    <resolution>0.1</resolution>
+                </range>
+                <noise>
+                    <type>gaussian</type>
+                    <mean>0.0</mean>
+                    <stddev>0.01</stddev>
+                </noise>
+            </ray>
+            <!--
+            <plugin name="lidar_sensor" filename="libgazebo_ros_ray_sensor.so">
+                <frameName>lidar_link</frameName>
+                <topicName>lidar/scan</topicName>
+                <updateRate>10.0</updateRate>
+                <visualize>true</visualize>
+            </plugin>
+            -->
+        </sensor>
+    </gazebo>
 </robot>
